File: sensorboard_18_v7.brd (EAGLE design)
At the start: 100 x 58 mm, 102 parts, among them IC2_ESP32S2WROOMM22S2 ESP32-S2-WROOM_M22S2H3200PH3Q0, IC4 TPA6211A1DRBR, J4_USB USB_CONN, J5_AUDIO SJ-3523-SMT-TR, J6_OAT 2.5mm JACK, J7 30310-6002HB, U1 LPS22HB, U10-MAG_SENSOR MMC5983MA, U11 LDL212PV33R, U12 NCV8163ASN330T1G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

Commit message: upload v18 files
Parts:
- removed AUDIO_SOURCE: (no value), pinhead:1X03
- removed FL1-USB_EMI: DLM0NSM900HY2D, SamacSys_Parts:DLM0NSB120HY2B
- added C30: 1uF, rcl:C0805
- added IC1: ECMF02-2AMX6, ECMF02-2AMX6:SON50P150X170X55-6N
- added R25: FERRITE, rcl:R0805
- added R26, R27: 10k, rcl:R0805
- C1, C11, C13, C16, C2, C3: value (none) -> 100nF
- C10, C29, C4, C41, C42, C5, C51, C52, C61, C62, C72, C8: value (none) -> 10uF
- C12: value (none) -> 10uF; device resistor:C0805 -> rcl:C0805
- C14, C15, C19, C27, C28, C6, C7, C9: value (none) -> 1uF
- C17, C18, C21, C22: value CL31A226KAHNNNE -> 22uF/25V
- C20: value (none) -> 47pF
- C23, C24: value (none) -> 470pF
- C25, C26: value (none) -> 220nF
- L1, L2, L3: value FDSD0420-H-100M=P3 -> 10uH
- R10, R14: value (none) -> 10k
- R11: value (none) -> 7k68
- R12: value (none) -> 75k
- R13: value (none) -> DNP
- R18, R19, R20, R21, R22, R3, R4, R5, R6, R7, R8: value (none) -> FERRITE
- R9: value (none) -> 40k2
- moved C21 19.6 mm to (27.6, 53.6)
- moved C18 11.8 mm to (15.9, 54.4), turned to 90 degrees
- moved C17 7.89 mm to (8.04, 53.7), turned to 270 degrees
- moved C29 1.40 mm to (81.1, 21.2)
- moved C25 1.08 mm to (82.3, 26.0)
- moved R17 0.62 mm to (72.6, 23.0), turned to 90 degrees
- moved R16 0.53 mm to (70.6, 23.0), turned to 90 degrees
- moved U$1 0.50 mm to (3.38, 8.75)
- moved R10 0.08 mm to (88.8, 34.9)
- renumbered AUD_DAUGHTER-B_IN to AUD_IN
Connections:
- removed net N$30: J4_USB.2, R16.2
- removed net N$31: J4_USB.3, R17.2
- new net 5V_AUD: AUD_IN.3, C28.1, C29.1, IC4.1, IC4.6, R25.2
- new net D+: IC1.6, J4_USB.3
- new net D-: IC1.5, J4_USB.2
- new net N$33: C20.1, C21.2, D2.2, L2.2, R9.2
- net 5VC: now also R25.1; no longer AUD_IN.3, C28.1, C29.1, IC4.1, IC4.6
- net 5VD: now also C30.1
- net AUD_IN: now also R26.1; no longer AUDIO_SOURCE.2, C25.1
- net ESP_AUD: now also R27.1; no longer AUDIO_SOURCE.3
- net GND: now also C30.2, IC1.3, U3-IMU.1; no longer AUDIO_SOURCE.1
- net N$13: now also C18.2; no longer C17.2
- net N$15: now also C25.1, R26.2, R27.2; no longer C18.2, C20.1, D2.2, L2.2, R9.2
- net N$27: now also IC1.1, R17.1; no longer FL1-USB_EMI.1, R16.1
- net N$28: now also IC1.2, R16.1; no longer FL1-USB_EMI.4, R17.1
- net N$9: now also C17.2; no longer C21.2
- net USB_D+: now also R16.2; no longer FL1-USB_EMI.3
- net USB_D-: now also R17.2; no longer FL1-USB_EMI.2
Routing:
- net GND: track 258.0 -> 211.3 mm, vias 598 -> 578
- net 5V_AUD: track 0.00 -> 44.1 mm, vias 0 -> 2
- net 5VC: track 163.1 -> 131.0 mm, vias 4 -> 3
- net N$33: track 0.00 -> 14.5 mm
- net N$30: track 13.1 -> 0.00 mm
- net N$31: track 11.7 -> 0.00 mm
- net N$15: track 15.5 -> 5.60 mm
- net D-: track 0.00 -> 6.71 mm
- net D+: track 0.00 -> 5.53 mm
- net AUD_IN: track 8.15 -> 2.77 mm
- net N$28: track 3.00 -> 6.69 mm
- net N$27: track 3.02 -> 6.57 mm
- net USB_D-: track 28.4 -> 31.0 mm
- net N$26: track 3.46 -> 5.53 mm
- net 5VD: track 111.0 -> 112.9 mm, vias 4 -> 5
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Other:
- board text added: "12V-GND"
- board text added: "DM/dD"
- board text added: "IN - GND - 5V"
- board text removed: "GND-IN-ESP_AUD"
- board text removed: "IN-GND-5V"
