File: sensorboard_18_v7.sch (EAGLE design)
At the start: 102 parts, among them IC2_ESP32S2WROOMM22S2 ESP32-S2-WROOM_M22S2H3200PH3Q0, IC4 TPA6211A1DRBR, J4_USB USB_CONN, J5_AUDIO SJ-3523-SMT-TR, J6_OAT 2.5mm JACK, J7 30310-6002HB, U1 LPS22HB, U10-MAG_SENSOR MMC5983MA, U11 LDL212PV33R, U12 NCV8163ASN330T1G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

Commit message: upload v18 files
Parts:
- removed AUDIO_SOURCE, AUD_DAUGHTER-B_IN: (no value), pinhead:PINHD-1X3
- removed FL1-USB_EMI: DLM0NSM900HY2D, SamacSys_Parts:DLM0NSM900HY2D
- added AUD_IN: (no value), pinhead:PINHD-1X3
- added C30: 1uF, rcl:C-EUC0805
- added IC1: ECMF02-2AMX6, ECMF02-2AMX6:ECMF02-2AMX6
- added R25: FERRITE, rcl:R-EU_R0805
- added R26, R27: 10k, rcl:R-EU_R0805
- C1, C11, C13, C16, C2, C3: value (none) -> 100nF
- C10, C29, C4, C41, C42, C5, C51, C52, C61, C62, C72, C8: value (none) -> 10uF
- C12: value (none) -> 10uF; device resistor:C-USC0805 -> rcl:C-EUC0805
- C14, C15, C19, C27, C28, C6, C7, C9: value (none) -> 1uF
- C17, C18, C21, C22: value CL31A226KAHNNNE -> 22uF/25V
- C20: value (none) -> 47pF
- C23, C24: value (none) -> 470pF
- C25, C26: value (none) -> 220nF
- L1, L2, L3: value FDSD0420-H-100M=P3 -> 10uH
- R10, R14: value (none) -> 10k
- R11: value (none) -> 7k68
- R12: value (none) -> 75k
- R13: value (none) -> DNP
- R18, R19, R20, R21, R22, R3, R4, R5, R6, R7, R8: value (none) -> FERRITE
- R9: value (none) -> 40k2
Connections:
- removed net N$30: J4_USB.2, R16.2
- removed net N$31: J4_USB.3, R17.2
- new net 5V_AUD: AUD_IN.3, C28.1, C29.1, IC4.!SHUTDOWN, IC4.VDD, R25.2
- new net D+: IC1.D+, J4_USB.3
- new net D-: IC1.D-, J4_USB.2
- new net N$33: C20.1, C21.2, D2.A, L2.2, R9.2
- net 5VC: now also R25.1; no longer AUD_DAUGHTER-B_IN.3, C28.1, C29.1, IC4.!SHUTDOWN, IC4.VDD
- net 5VD: now also C30.1
- net AUD_IN: now also AUD_IN.1, R26.1; no longer AUDIO_SOURCE.2, AUD_DAUGHTER-B_IN.1, C25.1
- net ESP_AUD: now also R27.1; no longer AUDIO_SOURCE.3
- net GND: now also AUD_IN.2, C30.2, U3-IMU.SDO/SA0; no longer AUDIO_SOURCE.1, AUD_DAUGHTER-B_IN.2
- net N$13: now also C18.2; no longer C17.2
- net N$15: now also C25.1, R26.2, R27.2; no longer C18.2, C20.1, D2.A, L2.2, R9.2
- net N$27: now also IC1.D_1, R17.1; no longer FL1-USB_EMI.1, R16.1
- net N$28: now also IC1.D_2, R16.1; no longer FL1-USB_EMI.4, R17.1
- net N$9: now also C17.2; no longer C21.2
- net USB_D+: now also R16.2; no longer FL1-USB_EMI.3
- net USB_D-: now also R17.2; no longer FL1-USB_EMI.2
Other:
- note added: "GAIN: 20k-2x 10k-4x"
- note added: "I2C address: 0110000"
- note added: "I2C address: 0x28 / 0101000"
- note added: "I2C address: 0x46H"
- note added: "I2C address: 0x78"
- note added: "I2C address: 1011100(bin) / 5C(hex)"
- note added: "I2C address: 1011101(bin) / 5D(hex)"
- note added: "I2C address: 1101010"
- moved on the sheet: C14, C15, C17, C18, C21, C24, L2, R10, R16, R17, R18, R19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
