File: archive/sensorboard_18_v7.sch (EAGLE design)
At the start: 90 parts, among them IC1 ECMF02-2AMX6, IC2_ESP32S2WROOMM22S2 ESP32-S2-WROOM_M22S2H3200PH3Q0, J1_CONN._ADAPTERB. RJ12, J4_USB USB_CONN, J6_OAT 2.5mm JACK, J7_I2C RJ12, U1 LPS22HB, U10-MAG_SENSOR MMC5983MA, U11 LDL212PV33R, U12 NCV8163ASN330T1G, U13-I2C DS2482S-100+, U2 LPS22HB, U3-IMU LSM6DSMTR, U4 NCV8163ASN330T1G, U5 NCV8163ASN330T1G, U6 NCV8163ASN330T1G, U7 NCV8163ASN330T1G

Commit message: Archive v18 files
Create archive directory with v18 files for use as assembly reference for previous board revision
Parts:
- removed ESP_AUD: (no value), pinhead:PINHD-1X2
- removed J1_CONN._ADAPTERB., J7_I2C: RJ12, Sensor_Board_DS2:SAMACSYS_615006138421"
- added AUD_DAUGHTER-B_OUT: (no value), pinhead:PINHD-1X2
- added AUD_IN: (no value), pinhead:PINHD-1X3
- added C24: 470pF, rcl:C-EUC0805
- added C25, C26: 220nF, rcl:C-EUC1206
- added C27, C28: 1uF, rcl:C-EUC1206
- added C29: 10uF, rcl:C-EUC1206
- added IC4: TPA6211A1DRBR, SamacSys_Parts:TPA6211A1DRBR
- added J5_AUDIO: SJ-3523-SMT-TR, SamacSys_Parts:SJ-3523-SMT-TR
- added J7: 30310-6002HB, SamacSys_Parts:30310-6002HB
- added OUTA, OUTB: (no value), wirepad_SMALL:SMD2_SMALLSMALL
- added R14, R26, R27: 10k, rcl:R-EU_R0805
- added R15: (no value), rcl:R-EU_R0805
- added R25: FERRITE, rcl:R-EU_R0805
- C23: value 100nF -> 470pF
- C71: value 10uF -> (none)
- D1: value SS24FL -> (none)
- R1, R2, R23, R24: value 10k -> (none)
- R16, R17: value FERRITE -> (none)
- U$4: value 4515DO-DS3BK030DPL -> (none)
- renumbered U$3 to DLHR-L30G-E1BD-C-NAV8
Connections:
- new net 5V_AUD: AUD_IN.3, C28.1, C29.1, IC4.!SHUTDOWN, IC4.VDD, R25.2
- new net AUD_IN: AUD_IN.1, R26.1
- new net AUD_OUT_A: AUD_DAUGHTER-B_OUT.1, C24.2, IC4.VO-, J5_AUDIO.SLEEVE, OUTA.P
- new net AUD_OUT_B: AUD_DAUGHTER-B_OUT.2, C23.2, IC4.VO+, J5_AUDIO.TIP, OUTB.P
- new net CLK: J7.9
- new net CS0: J7.10
- new net CS1: J7.4
- new net MISO: J7.7
- new net MOSI: J7.8
- new net N$15: C25.1, R26.2, R27.2
- new net N$21: C24.1, IC4.IN+, R14.2
- new net N$22: C26.2, R14.1
- new net N$23: C25.2, R15.1
- new net N$26: C27.1, IC4.BYPASS
- new net N$8: C23.1, IC4.IN-, R15.2
- net 3V3: now also J7.1; no longer J1_CONN._ADAPTERB..2
- net 3V3_DIG: no longer J7_I2C.2
- net 5VC: now also R25.1; no longer J7_I2C.1
- net 5V_EXT: now also J7.3; no longer J1_CONN._ADAPTERB..1
- net ESP_AUD: now also R27.1; no longer ESP_AUD.1
- net GND: now also AUD_IN.2, C26.1, C27.2, C28.2, C29.2, IC4.EP_1, IC4.EP_2, IC4.EP_3, IC4.EP_4, IC4.EP_5, IC4.GND, J5_AUDIO.RING, J7.2; no longer C23.2, ESP_AUD.2, J1_CONN._ADAPTERB..5, J1_CONN._ADAPTERB..6, J7_I2C.5, J7_I2C.6
- net N$7: no longer C23.1
- net SCL0: no longer J7_I2C.4
- net SCL1: now also J7.5; no longer J1_CONN._ADAPTERB..4
- net SDA0: no longer J7_I2C.3
- net SDA1: now also J7.6; no longer J1_CONN._ADAPTERB..3
Other:
- note added: "GAIN: 20k-2x 10k-4x"
- note removed: "DNP=Do Not Populate"
- note removed: "FERRITES: MI0805K601R-10"
- moved on the sheet: C23, D3, J6_OAT, R10
